Commit message: modifie urdf model

File: p3at_description/urdf/pioneer3at.urdf.xacro (robot description, xacro)
@@ -6,12 +6,14 @@
   xmlns:xacro="http://ros.org/wiki/xacro"
   name="pioneer3at">
-  <xacro:include filename="$(find p3at_description)/urdf/pioneer3at_body.xacro"/>
-  <xacro:include filename="$(find p3at_description)/urdf/hokuyo_utm30lx.urdf.xacro"/>
-  <xacro:include filename="$(find p3at_description)/urdf/asus_camera.urdf.xacro" />
- <xacro:hokuyo_utm30lx name="hokuyo" parent="base_link" ros_topic="hokuyo" update_rate="25" ray_count="720" min_angle="130" max_angle="-130">
-    <origin xyz="0.13 0 0.32" rpy="0 0 0"/>
-  </xacro:hokuyo_utm30lx>
-  <xacro:asus_camera name="camera" parent="base_link">
-	  <origin xyz="0.065 0.0 0.43" rpy="0 0 0"/>
-  </xacro:asus_camera>
+{
+    <xacro:include filename="$(find p3at_description)/urdf/pioneer3at_body.xacro"/>
+    <xacro:include filename="$(find p3at_description)/urdf/hokuyo_utm30lx.urdf.xacro"/>
+    <xacro:include filename="$(find p3at_description)/urdf/asus_camera.urdf.xacro" />
+  </xacro:macro>
+   <xacro:hokuyo_utm30lx name="hokuyo" parent="base_link" ros_topic="hokuyo" update_rate="25" ray_count="720" min_angle="130" max_angle="-130">
+      <origin xyz="0.13 0 0.32" rpy="0 0 0"/>
+    </xacro:hokuyo_utm30lx>
+    <xacro:asus_camera name="camera" parent="base_link">
+  	  <origin xyz="0.065 0.0 0.43" rpy="0 0 0"/>
+    </xacro:asus_camera>
 </robot>

Commit message: Revert a wrong commit

File: p3at_description/urdf/pioneer3at.urdf.xacro (robot description, xacro)
@@ -6,14 +6,12 @@
   xmlns:xacro="http://ros.org/wiki/xacro"
   name="pioneer3at">
-{
-    <xacro:include filename="$(find p3at_description)/urdf/pioneer3at_body.xacro"/>
-    <xacro:include filename="$(find p3at_description)/urdf/hokuyo_utm30lx.urdf.xacro"/>
-    <xacro:include filename="$(find p3at_description)/urdf/asus_camera.urdf.xacro" />
-  </xacro:macro>
-   <xacro:hokuyo_utm30lx name="hokuyo" parent="base_link" ros_topic="hokuyo" update_rate="25" ray_count="720" min_angle="130" max_angle="-130">
-      <origin xyz="0.13 0 0.32" rpy="0 0 0"/>
-    </xacro:hokuyo_utm30lx>
-    <xacro:asus_camera name="camera" parent="base_link">
-  	  <origin xyz="0.065 0.0 0.43" rpy="0 0 0"/>
-    </xacro:asus_camera>
+  <xacro:include filename="$(find p3at_description)/urdf/pioneer3at_body.xacro"/>
+  <xacro:include filename="$(find p3at_description)/urdf/hokuyo_utm30lx.urdf.xacro"/>
+  <xacro:include filename="$(find p3at_description)/urdf/asus_camera.urdf.xacro" />
+  <xacro:hokuyo_utm30lx name="hokuyo" parent="base_link" ros_topic="hokuyo" update_rate="25" ray_count="720" min_angle="130" max_angle="-130">
+    <origin xyz="0.13 0 0.32" rpy="0 0 0"/>
+  </xacro:hokuyo_utm30lx>
+  <xacro:asus_camera name="camera" parent="base_link">
+    <origin xyz="0.065 0.0 0.43" rpy="0 0 0"/>
+  </xacro:asus_camera>
 </robot>
